File: pork pi.sch (EAGLE design)
At the start: 116 parts, among them J1 SJ-2523-SMT-TR, J3 MICRO-SD, U1 A13, U2 AXP209, U3 AP2161DM8G-13, U4 HC-05, Y1 24MHz

Commit message: Schematic update
Added 3.3V and 1.5V ddr3 switching regulators and all necessary
inductors and other passives.
Parts:
- added C65, C71, C73, C74, C76, C77, C78, C81: 22uF, SparkFun-Passives:CAP0603-CAP
- added C66, C72, C75, C79, C82: 0.1uF, SparkFun-Passives:CAP0402-CAP
- added C67, C68: 1nF, SparkFun-Passives:CAP0402-CAP
- added C69, C70: 22pF, SparkFun-Passives:CAP0402-CAP
- added C80: 10uF, SparkFun-Passives:CAP0603-CAP
- added D2: 1N4148W-TP, Passives:DIODE
- added D3: B340-13-F, Diodes:B340-13-F
- added J4: POWER_JACKPTH, SparkFun-Connectors:POWER_JACKPTH
- added JP2: JUMPER-31-2, SparkFun-Passives:JUMPER-31-2
- added L5: NR6028T220M, Taiyo Yuden:NR6028T4R7M
- added L6, L7, L8: NR6028T2R2N, Taiyo Yuden:NR6028T4R7M
- added PT1, PT2, PT3, PT4: 2PT_GND_TIE, SparkFun-Passives:2PT_GND_TIE
- added Q1: DMP3098L-7, Diodes:DMP3098L-7
- added R31: 100kΩ, SparkFun-Passives:RESISTOR0402-RES
- added R32, R35, R39, R41: 33kΩ, SparkFun-Passives:RESISTOR0402-RES
- added R33, R37: 330kΩ, SparkFun-Passives:RESISTOR0402-RES
- added R34, R38: 30kΩ, SparkFun-Passives:RESISTOR0402-RES
- added R36: 37kΩ, SparkFun-Passives:RESISTOR0402-RES
- added R40: 10.5kΩ, SparkFun-Passives:RESISTOR0402-RES
- added R42: 6.2kΩ, SparkFun-Passives:RESISTOR0402-RES
- added U5: MIC2250YML, Micrel:MIC2250YML
- added U6, U7: AP3409DNTR-G1, Diodes:AP3409DNTR-G1
- added U8: ST1S10PUR, STMicroelectrionics:ST1S10PUR
Connections:
- new net FGND: PT1.P$2, PT2.P$2, PT3.P$2, PT4.P$2, U5.PGND, U6.PGND, U7.PGND, U8.PGND
- new net N$37: JP2.2, U5.DITH
- new net N$38: D2.P$1, L5.2, U5.SW
- new net N$39: R31.1, R32.2, U5.FB
- new net N$40: C65.1, C66.1, D2.P$2, Q1.D, R31.2
- new net N$42: R33.2, U6.SHDN/RT
- new net N$43: C67.1, R34.1
- new net N$44: R34.2, U6.COMP
- new net N$45: R37.2, U7.SHDN/RT
- new net N$46: C68.1, R38.1
- new net N$47: R38.2, U7.COMP
- new net N$48: L7.1, U7.SW
- new net N$49: C79.1, C80.1, J4.PWR, U8.EN, U8.VIN_A, U8.VIN_SW
- new net N$50: C69.1, R39.1, R40.2, U7.FB
- new net N$51: L6.1, U6.SW
- new net N$52: L8.1, U8.SW
- new net N$53: C70.1, R35.1, R36.2, U6.FB
- new net N$54: C81.1, C82.1, D3.A, L8.2, Q1.G, R41.2
- new net N$55: R41.1, R42.2, U8.FB
- net 1.5V_DDR: now also C74.1, C75.1, C76.1, L6.2, R35.2
- net 3.3V: now also C71.1, C72.1, C73.1, L7.2, R39.2
- net 5V: now also D3.C, Q1.S
- net GND: now also C65.2, C66.2, C67.2, C68.2, C69.2, C70.2, C71.2, C72.2, C73.2, C74.2, C75.2, C76.2, C77.2, C78.2, C79.2, C80.2, C81.2, C82.2, J4.GND, J4.GNDBREAK, JP2.1, PT1.P$1, PT2.P$1, PT3.P$1, PT4.P$1, R32.1, R33.1, R36.1, R37.1, R40.1, R42.1, U5.AGND, U6.GND, U7.GND, U8.AGND, U8.SYNC
- net IPSOUT: now also C77.1, C78.1, JP2.3, L5.1, U5.EN, U5.VIN, U6.PVDD, U6.VDD, U7.PVDD, U7.VDD
Other:
- note added: "R2 = R1 / ((Vout / 1.24) - 1)"
- note added: "Vout = 0.8 * (1 + R1/R2)"
- note added: "Vout = 0.8 * (R1 + R2) / R2"
- moved on the sheet: C14, C15, C2, C22, C23, C24, C27, C3, J2, JP1, R13, R14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

Commit message: Schematic update
Added SK HYNIX 2Gb DD3 chips and necessary signals
Parts:
- added C83, C84, C85, C86, C87, C88, C89, C90, C91, C92, C94, C95, C96, C97, C98: 0.1uF, SparkFun-Passives:CAP0402-CAP
- added C93, C99: 22uF, SparkFun-Passives:CAP0603-CAP
- added R43, R50: 240Ω 1%, SparkFun-Passives:RESISTOR0402-RES
- added R44, R45: 2kΩ 1%, SparkFun-Passives:RESISTOR0402-RES
- added R46, R47, R48, R49: 22Ω, SparkFun-Passives:RESISTOR0402-RES
- added RN1, RN10, RN11, RN2, RN3, RN4, RN5, RN6, RN7, RN8, RN9: 22Ω, Passives:RESISTOR-NETWORK-1206
- added U$4, U$5: DDR3, SK HYNIX:DDR3
Connections:
- new net !DDR3_CAS!: RN9A.1, U$4.!CAS, U$5.!CAS
- new net !DDR3_RAS!: RN9B.1, U$4.!RAS, U$5.!RAS
- new net !DDR3_WE!: RN5D.1, U$4.!WE, U$5.!WE
- new net DDR3_A0: RN5A.1, U$4.A0, U$5.A0
- new net DDR3_A1: RN6C.1, U$4.A1, U$5.A1
- new net DDR3_A10: RN7C.1, U$4.A10/AP, U$5.A10/AP
- new net DDR3_A11: RN9D.1, U$4.A11, U$5.A11
- new net DDR3_A12: RN7A.1, U$4.A12/!BC, U$5.A12/!BC
- new net DDR3_A13: RN8A.1, U$4.A13, U$5.A13
- new net DDR3_A14: RN9C.1, U$4.A14, U$5.A14
- new net DDR3_A2: RN8C.1, U$4.A2, U$5.A2
- new net DDR3_A3: RN8D.1, U$4.A3, U$5.A3
- new net DDR3_A4: RN6D.1, U$4.A4, U$5.A4
- new net DDR3_A5: RN8B.1, U$4.A5, U$5.A5
- new net DDR3_A6: RN6B.1, U$4.A6, U$5.A6
- new net DDR3_A7: RN10B.1, U$4.A7, U$5.A7
- new net DDR3_A8: RN6A.1, U$4.A8, U$5.A8
- new net DDR3_A9: RN10D.1, U$4.A9, U$5.A9
- new net DDR3_BA0: RN5B.1, U$4.BA0, U$5.BA0
- new net DDR3_BA1: RN7B.1, U$4.BA1, U$5.BA1
- new net DDR3_BA2: RN5C.1, U$4.BA2, U$5.BA2
- new net DDR3_CKE: RN7D.1, U$4.CKE, U$5.CKE
- new net DDR3_CK_N: R47.1, U$4.!CK, U$5.!CK
- new net DDR3_CK_P: R46.1, U$4.CK, U$5.CK
- new net DDR3_D0: RN1A.1, U$4.DQ0
- new net DDR3_D1: RN3D.1, U$4.DQ1
- new net DDR3_D10: RN2A.1, U$5.DQ5
- new net DDR3_D11: RN4D.1, U$5.DQ4
- new net DDR3_D12: RN2D.1, U$5.DQ1
- new net DDR3_D13: RN4B.1, U$5.DQ2
- new net DDR3_D14: RN2B.1, U$5.DQ7
- new net DDR3_D15: RN4A.1, U$5.DQ0
- new net DDR3_D2: RN1B.1, U$4.DQ2
- new net DDR3_D3: RN3C.1, U$4.DQ3
- new net DDR3_D4: RN1D.1, U$4.DQ4
- new net DDR3_D5: RN3A.1, U$4.DQ5
- new net DDR3_D6: RN1C.1, U$4.DQ6
- new net DDR3_D7: RN3B.1, U$4.DQ7
- new net DDR3_D8: RN2C.1, U$5.DQ3
- new net DDR3_D9: RN4C.1, U$5.DQ6
- new net DDR3_DM0: R48.1, U$4.DM/TDQS
- new net DDR3_DM1: R49.1, U$5.DM/TDQS
- new net DDR3_DQS0_N: RN11C.1, U$4.!DQS
- new net DDR3_DQS0_P: RN11D.1, U$4.DQS
- new net DDR3_DQS1_N: RN11A.1, U$5.!DQS
- new net DDR3_DQS1_P: RN11B.1, U$5.DQS
- new net DDR3_ODT: RN10A.1, U$4.ODT, U$5.ODT
- new net DDR3_RST: RN10C.1, U$4.!RESET, U$5.!RESET
- new net DDR_VREF: C84.1, C85.1, C87.1, C88.1, R44.2, R45.1, U$4.VREFCA, U$4.VREFDQ, U$5.VREFCA, U$5.VREFDQ
- new net N$100: R46.2, U1D.DDR3_CK+
- new net N$101: R47.2, U1D.DDR3_CK-
- new net N$102: R49.2, U1D.DDR3_DM1
- new net N$103: R48.2, U1D.DDR3_DM0
- new net N$104: R50.2, U$5.ZQ
- new net N$41: R43.2, U$4.ZQ
- new net N$56: RN1A.2, U1D.DDR3_D0
- new net N$57: RN1B.2, U1D.DDR3_D2
- new net N$58: RN1D.2, U1D.DDR3_D4
- new net N$59: RN1C.2, U1D.DDR3_D6
- new net N$60: RN2A.2, U1D.DDR3_D10
- new net N$61: RN2B.2, U1D.DDR3_D14
- new net N$62: RN2C.2, U1D.DDR3_D8
- new net N$63: RN2D.2, U1D.DDR3_D12
- new net N$64: RN3D.2, U1D.DDR3_D1
- new net N$65: RN3C.2, U1D.DDR3_D3
- new net N$66: RN3A.2, U1D.DDR3_D5
- new net N$67: RN3B.2, U1D.DDR3_D7
- new net N$68: RN4B.2, U1D.DDR3_D13
- new net N$69: RN4A.2, U1D.DDR3_D15
- new net N$70: RN4D.2, U1D.DDR3_D11
- new net N$71: RN4C.2, U1D.DDR3_D9
- new net N$72: RN5A.2, U1D.DDR3_A0
- new net N$73: RN5B.2, U1D.DDR3_BA0
- new net N$74: RN5C.2, U1D.DDR3_BA2
- new net N$75: RN5D.2, U1D.DDR3_WE
- new net N$76: RN6A.2, U1D.DDR3_A8
- new net N$77: RN6B.2, U1D.DDR3_A6
- new net N$78: RN6D.2, U1D.DDR3_A4
- new net N$79: RN6C.2, U1D.DDR3_A1
- new net N$80: RN7D.2, U1D.DDR3_CKE
- new net N$81: RN7A.2, U1D.DDR3_A12
- new net N$82: RN7C.2, U1D.DDR3_A10
- new net N$83: RN7B.2, U1D.DDR3_BA1
- new net N$84: RN8C.2, U1D.DDR3_A2
- new net N$85: RN8D.2, U1D.DDR3_A3
- new net N$86: RN8B.2, U1D.DDR3_A5
- new net N$87: RN8A.2, U1D.DDR3_A13
- new net N$88: RN9D.2, U1D.DDR3_A11
- new net N$89: RN9C.2, U1D.DDR3_A14
- new net N$90: RN9B.2, U1D.DDR3_RAS
- new net N$91: RN9A.2, U1D.DDR3_CAS
- new net N$92: RN10B.2, U1D.DDR3_A7
- new net N$93: RN10D.2, U1D.DDR3_A9
- new net N$94: RN10C.2, U1D.DDR3_RST
- new net N$95: RN10A.2, U1D.DDR3_ODT
- new net N$96: RN11D.2, U1D.DDR3_DQS0+
- new net N$97: RN11C.2, U1D.DDR3_DQS0-
- new net N$98: RN11B.2, U1D.DDR3_DQS1+
- new net N$99: RN11A.2, U1D.DDR3_DQS1-
- net 1.5V_DDR: now also C83.1, C86.1, C89.1, C90.1, C91.1, C92.1, C93.1, C94.1, C95.1, C96.1, C97.1, C98.1, C99.1, R45.2, U$4.VDD@1, U$4.VDD@2, U$4.VDD@3, U$4.VDD@4, U$4.VDD@5, U$4.VDD@6, U$4.VDD@7, U$4.VDD@8, U$4.VDD@9, U$4.VDDQ@1, U$4.VDDQ@2, U$4.VDDQ@3, U$4.VDDQ@4, U$5.VDD@1, U$5.VDD@2, U$5.VDD@3, U$5.VDD@4, U$5.VDD@5, U$5.VDD@6, U$5.VDD@7, U$5.VDD@8, U$5.VDD@9, U$5.VDDQ@1, U$5.VDDQ@2, U$5.VDDQ@3, U$5.VDDQ@4
- net GND: now also C83.2, C84.2, C85.2, C86.2, C87.2, C88.2, C89.2, C90.2, C91.2, C92.2, C93.2, C94.2, C95.2, C96.2, C97.2, C98.2, C99.2, R43.1, R44.1, R50.1, U$4.!CS, U$4.VSS@1, U$4.VSS@10, U$4.VSS@11, U$4.VSS@12, U$4.VSS@2, U$4.VSS@3, U$4.VSS@4, U$4.VSS@5, U$4.VSS@6, U$4.VSS@7, U$4.VSS@8, U$4.VSS@9, U$4.VSSQ@1, U$4.VSSQ@2, U$4.VSSQ@3, U$4.VSSQ@4, U$4.VSSQ@5, U$5.!CS, U$5.VSS@1, U$5.VSS@10, U$5.VSS@11, U$5.VSS@12, U$5.VSS@2, U$5.VSS@3, U$5.VSS@4, U$5.VSS@5, U$5.VSS@6, U$5.VSS@7, U$5.VSS@8, U$5.VSS@9, U$5.VSSQ@1, U$5.VSSQ@2, U$5.VSSQ@3, U$5.VSSQ@4, U$5.VSSQ@5
Other:
- moved on the sheet: U1D

Commit message: Schematic Update
Added HDMI controller and required components
Parts:
- added C100, C101, C102, C103, C104, C105, C106: 0.1uF, SparkFun-Passives:CAP0402-CAP
- added C107: 120uF, Passives:CAP_POL-POLYMER_6.5
- added J5: HDMI-SMD, FCI:HDMI-SMD
- added PT5: 2PT_GND_TIE, SparkFun-Passives:2PT_GND_TIE
- added R51: 10kΩ, SparkFun-Passives:RESISTOR0402-RES
- added RN12: 22Ω, Passives:RESISTOR-NETWORK-1206
- added U9: TFP410, TI:TFP410
- R10: value 22Ω -> 10kΩ
- R11: value 22Ω -> 1.2kΩ
- R9: value 22Ω -> 470Ω
Connections:
- new net CEC: J5.CEC, U1I.PB3/EINT17
- new net HTPLG: J5.HOTPLUG, R11.1
- new net MSEN: R51.1, U1I.PB2/EINT16, U9A.MSEN/PO1
- new net N$105: U1H.LCD_D23, U9C.D23
- new net N$106: U1H.LCD_D22, U9C.D22
- new net N$107: U1H.LCD_D21, U9C.D21
- new net N$108: U1H.LCD_D20, U9C.D20
- new net N$109: U1H.LCD_D19, U9C.D19
- new net N$110: U1H.LCD_D18, U9C.D18
- new net N$111: U1H.LCD_D15, U9C.D15
- new net N$112: U1H.LCD_D14, U9C.D14
- new net N$113: U1H.LCD_D13, U9C.D13
- new net N$114: U1H.LCD_D12, U9C.D12
- new net N$115: U1H.LCD_D11, U9C.D11
- new net N$116: U1H.LCD_D10, U9C.D10
- new net N$117: U1H.LCD_D7, U9C.D7
- new net N$118: U1H.LCD_D6, U9C.D6
- new net N$119: U1H.LCD_D5, U9C.D5
- new net N$120: U1H.LCD_D4, U9C.D4
- new net N$121: U1H.LCD_D3, U9C.D3
- new net N$122: U1H.LCD_D2, U9C.D2
- new net N$123: U1H.LCD_CLK, U9C.IDCK+
- new net N$124: U1H.LCD_DE, U9C.DE
- new net N$125: U1H.LCD_HSYNC, U9C.HSYNC
- new net N$126: U1H.LCD_VSYNC, U9C.VSYNC
- new net N$127: R9.1, U9A.TFADJ
- new net N$128: R10.1, U9A.ISEL/!RST
- new net N$129: R11.2, U9A.EDGE/HTPLG
- new net N$130: J5.TX2+, U9B.TX2+
- new net N$131: J5.TX2-, U9B.TX2-
- new net N$132: J5.TX1+, U9B.TX1+
- new net N$133: J5.TX1-, U9B.TX1-
- new net N$134: J5.TX0+, U9B.TX0+
- new net N$135: J5.TX0-, U9B.TX0-
- new net N$136: J5.TXC+, U9B.TXC+
- new net N$137: J5.TXC-, U9B.TXC-
- net 3.3V: now also C100.1, C101.1, C102.1, C103.1, C104.1, C105.1, C106.1, R10.2, R51.2, R9.2, U9A.DVDD@1, U9A.DVDD@2, U9A.DVDD@3, U9A.PVDD@1, U9A.TVDD@1, U9A.TVDD@2, U9A.VREF
- net 5V: now also J5.5V
- net FGND: now also J5.SHIELD, PT5.P$2
- net GND: now also C100.2, C101.2, C102.2, C103.2, C104.2, C105.2, C106.2, C107.-, J5.GND, J5.TGND@1, J5.TGND@2, J5.TGND@3, J5.TGND@4, PT5.P$1, U9A.!PD, U9A.CTL1/A1/DK1, U9A.CTL2/A2/DK2, U9A.CTL3/A3/DK3, U9A.DGND@1, U9A.DGND@2, U9A.DGND@3, U9A.DKEN, U9A.EP, U9A.PGND@1, U9A.RESERVED, U9A.TGND@1, U9A.TGND@2, U9A.TGND@3, U9C.D0, U9C.D1, U9C.D16, U9C.D17, U9C.D8, U9C.D9, U9C.IDCK-
- net N$10: now also RN12C.2; no longer R11.2
- net N$11: now also RN12A.1; no longer R9.1
- net N$12: now also RN12B.1; no longer R10.1
- net N$13: now also RN12C.1; no longer R11.1
- net N$49: now also C107.+
- net N$8: now also RN12A.2; no longer R9.2
- net N$9: now also RN12B.2; no longer R10.2
- net SCL: now also J5.SCL, U9A.BSEL/SCL
- net SDA: now also J5.SDA, U9A.DSEL/SDA
Other:
- moved on the sheet: C10, C11, C14, C15, C35, C36, C37, C38, C39, C40, C41, C42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

Commit message: Schematic update
Added NAND flash and all required signals. Also did a bit of rearranging
and fencing of different gates.
Parts:
- added C108, C109: 22pF, SparkFun-Passives:CAP0402-CAP
- added C110: 10uF, SparkFun-Passives:CAP0603-CAP
- added C111, C112, C114, C115, C116, C117, C118: 0.1uF, SparkFun-Passives:CAP0402-CAP
- added C113, C119: 22uF, SparkFun-Passives:CAP0603-CAP
- added J6: RB1-125BAG1A, Connectors:RB1-125BAG1A
- added J7: USB+SHIELD-MICROB, SparkFun-Connectors:USB+SHIELD-MICROB
- added JP3: (no value), SparkFun-Connectors:M04PTH
- added L9: 600Ω 0.5A, SparkFun-Passives:INDUCTOR0805
- added PT6, PT7: 2PT_GND_TIE, SparkFun-Passives:2PT_GND_TIE
- added R52, R53, R60, R61, R62: 10kΩ, SparkFun-Passives:RESISTOR0402-RES
- added R54, R55: 100Ω, SparkFun-Passives:RESISTOR0402-RES
- added R56, R57, R58, R59: 49.9Ω, SparkFun-Passives:RESISTOR0805-RES
- added U10: ENC28J60-QFN, Microchip:ENC28J60-QFN
- added U11: NAND, Samsung:NAND
- added U12: TUSB2077, TI:TUSB2077
- added U19, U20, U21: IP4220CZ6, NXP:IP4220CZ6
- added Y2: 25MHz, Passives:CRYSTAL-3.2X2.5
Connections:
- new net !ETH_INT: U10.!INT, U1I.PB4/EINT18
- new net D0_N: J7.D-, U1N.D0-
- new net D0_P: J7.D+, U1N.D0+
- new net N$138: C109.1, U10.OSC1, Y2.2
- new net N$139: C108.1, U10.OSC2, Y2.1
- new net N$140: R52.2, U10.RBIAS
- new net N$141: C110.1, U10.VCAP
- new net N$142: R53.1, U10.!RESET
- new net N$143: J6GREEN.C, R55.1
- new net N$144: J6YELLOW.C, R54.1
- new net N$145: J6GREEN.A, U10.LEDA
- new net N$146: J6YELLOW.A, U10.LEDB
- new net N$147: J6A.R1, R58.1, U10.TPOUT+
- new net N$148: J6A.R2, R59.1, U10.TPOUT-
- new net N$149: J6A.R7, R56.2, U10.TPIN+
- new net N$150: J6A.R8, R57.2, U10.TPIN-
- new net N$151: C111.1, J6A.R3, L9.1, R58.2, R59.2
- new net N$152: U11.D0, U1E.!DQ0!/SDC2_D0
- new net N$153: U11.D1, U1E.!DQ1!/SDC2_D1
- new net N$154: U11.D2, U1E.!DQ2!/SDC2_D2
- new net N$155: U11.D3, U1E.!DQ3!/SDC2_D3
- new net N$156: U11.D4, U1E.!DQ4!/SDC2_D4
- new net N$157: U11.D5, U1E.!DQ5!/SDC2_D5
- new net N$158: U11.D6, U1E.!DQ6!/SDC2_D6
- new net N$159: U11.D7, U1E.!DQ7!/SDC2_D7
- new net N$160: R60.1, U11.R/!B, U1E.!RB0!/SDC2_CMD
- new net N$161: R61.1, U11.!CE, U1E.!CE0
- new net N$162: U11.!WE, U1E.!WE!/SPI0_MOSI
- new net N$163: U11.!RE, U1E.!RE
- new net N$164: U11.ALE, U1E.!ALE!/SPI0_MISO
- new net N$165: U11.CLE, U1E.!CLE!/SPI0_CLK
- new net N$166: C112.1, R62.1, U11.!WP
- new net N$167: JP3.1, U1F.TPY1
- new net N$168: JP3.2, U1F.TPX1
- new net N$169: JP3.3, U1F.TPY2
- new net N$170: JP3.4, U1F.TPX2
- net 3.3V: now also C113.1, C114.1, C115.1, C116.1, C117.1, C118.1, C119.1, L9.2, R53.2, R60.2, R61.2, R62.2, U10.VDD, U10.VDDOSC, U10.VDDPLL, U10.VDDRX, U10.VDDTX, U11.VCC@1, U11.VCC@2
- net ETH_CLK: now also U10.SCK
- net ETH_CS: now also U10.!CS
- net ETH_MISO: now also U10.SO
- net ETH_MOSI: now also U10.SI
- net FGND: now also J6A.S$1, J6A.S$2, J7.P$1, J7.P$2, PT6.P$2, PT7.P$2
- net GND: now also C108.2, C109.2, C110.2, C111.2, C112.2, C113.2, C114.2, C115.2, C116.2, C117.2, C118.2, C119.2, J7.GND, PT6.P$1, PT7.P$1, R52.1, R54.2, R55.2, R56.1, R57.1, U10.VSS, U10.VSSOSC, U10.VSSPLL, U10.VSSRX, U10.VSSTX, U11.VSS@1, U11.VSS@2, Y2.GND
- net VUSB: now also J7.VBUS
Other:
- moved on the sheet: C10, C100, C101, C102, C103, C104, C105, C106, C107, C11, C12, C13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

Commit message: Schematic update
Added HC-05-EZ part as well as the USB hub and necessary connectors etc.
Parts:
- added C120, C121, C122, C123, C124, C125: 120uF, Passives:CAP_POL-POLYMER_6.5
- added C126, C127, C128: 1uF, SparkFun-Passives:CAP0402-CAP
- added C129, C130: 22pF, SparkFun-Passives:CAP0402-CAP
- added J8, J9: USB-STACKED, Connectors:USB-STACKED
- added PT8, PT9: 2PT_GND_TIE, SparkFun-Passives:2PT_GND_TIE
- added R63, R64, R65, R66, R67, R68: 22Ω, SparkFun-Passives:RESISTOR0402-RES
- added R69: 1.5kΩ, SparkFun-Passives:RESISTOR0402-RES
- added RN13, RN14, RN15: 22Ω, Passives:RESISTOR-NETWORK-1206
- added U13: HC-05-EZ, Passives:HC-05-EZ
- added U14, U15, U16: TPS2042, TI:TPS2042
- added Y3: 6MHz, Passives:CRYSTAL-3.2X2.5
Connections:
- new net BT_KEY: U13.KEY, U1I.PB15, U4.PIO11
- new net BT_LED: U13.LED, U1I.PB16
- new net D1_N: R68.1, U1M.D1-
- new net D1_P: R67.1, U1M.D1+
- new net D2_N: RN13A.1, U12B.DM1, U19.D0-
- new net D2_P: RN13B.1, U12B.DP1, U19.D0+
- new net D3_N: RN13C.1, U12C.DM2, U19.D1-
- new net D3_P: RN13D.1, U12C.DP2, U19.D1+
- new net D4_N: RN14A.1, U12D.DM3, U20.D0-
- new net D4_P: RN14B.1, U12D.DP3, U20.D0+
- new net D5_N: RN14C.1, U12E.DM4, U20.D1-
- new net D5_P: RN14D.1, U12E.DP4, U20.D1+
- new net D6_N: RN15A.1, U12F.DM5, U21.D0-
- new net D6_P: RN15B.1, U12F.DP5, U21.D0+
- new net D7_N: RN15C.1, U12G.DM6, U21.D1-
- new net D7_P: RN15D.1, U12G.DP6, U21.D1+
- new net N$171: U12B.!PWRON1, U14A.!EN
- new net N$172: U12B.!OVRCUR1, U14A.!OC
- new net N$173: J9C.D-, RN15C.2
- new net N$174: J9C.D+, RN15D.2
- new net N$175: J9B.D-, RN15A.2
- new net N$176: J9B.D+, RN15B.2
- new net N$177: J9A.D+, RN14D.2
- new net N$178: J9A.D-, RN14C.2
- new net N$179: U12D.!PWRON3, U15A.!EN
- new net N$180: U12D.!OVRCUR3, U15A.!OC
- new net N$181: U12C.!PWRON2, U14B.!EN
- new net N$182: U12C.!OVRCUR2, U14B.!OC
- new net N$183: C121.+, J8B.VBUS, U14B.OUT
- new net N$184: C120.+, J8A.VBUS, U14A.OUT
- new net N$185: C122.+, J8C.VBUS, U15A.OUT
- new net N$186: J8C.D+, RN14B.2
- new net N$187: J8C.D-, RN14A.2
- new net N$188: U12E.!OVRCUR4, U15B.!OC
- new net N$189: U12E.!PWRON4, U15B.!EN
- new net N$190: C123.+, J9A.VBUS, U15B.OUT
- new net N$191: J8B.D+, RN13D.2
- new net N$192: J8B.D-, RN13C.2
- new net N$193: U12F.!PWRON5, U16A.!EN
- new net N$194: U12F.!OVRCUR5, U16A.!OC
- new net N$195: C124.+, J9B.VBUS, U16A.OUT
- new net N$196: J8A.D+, RN13B.2
- new net N$197: J8A.D-, RN13A.2
- new net N$198: C125.+, J9C.VBUS, U16B.OUT
- new net N$199: U12G.!PWRON6, U16B.!EN
- new net N$200: U12G.!OVRCUR6, U16B.!OC
- new net N$201: C130.1, U12A.XTAL2, Y3.2
- new net N$202: C129.1, U12A.XTAL1, Y3.1
- new net N$203: J7.D+, R65.2
- new net N$204: J7.D-, R66.2
- new net N$205: R67.2, R69.1, U12A.DP0
- new net N$206: R68.2, U12A.DM0
- new net N$207: R69.2, U12A.DP0PUR
- net !RESET: now also U12A.!RESET
- net 3.3V: now also U12A.!BUSPWR, U12A.!EXTMEM, U12A.EEDATA, U12A.VCC@1, U12A.VCC@2, U13.VCC
- net 5V: now also C126.1, C127.1, C128.1, U14A.VCC, U15A.VCC, U16A.VCC, U19.VCC, U20.VCC, U21.VCC
- net D0_N: now also R66.1; no longer J7.D-
- net D0_P: now also R65.1; no longer J7.D+
- net FGND: now also J8A.P$1, J8A.P$2, J9A.P$1, J9A.P$2, PT8.P$2, PT9.P$2
- net GND: now also C120.-, C121.-, C122.-, C123.-, C124.-, C125.-, C126.2, C127.2, C128.2, C129.2, C130.2, J8A.GND, J8B.GND, J8C.GND, J9A.GND, J9B.GND, J9C.GND, PT8.P$1, PT9.P$1, U12A.GND@1, U12A.GND@2, U12A.GND@3, U12A.MODE, U13.GND, U14A.GND, U15A.GND, U16A.GND, U19.GND, U20.GND, U21.GND, Y3.GND
- net UART1_RX: now also U13.TX
- net UART1_TX: now also U13.RX
Other:
- moved on the sheet: C10, C11, C12, C13, R15, R16, R17, U19, U1M, U1N, U20, U21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
